File: hardware/nssfc.kicad_pcb (KiCad board)
At the start: 4 copper layers, 37 x 37 mm, 64 parts, among them J1 USB_C_Receptacle_USB2.0_16P, SW1 SW_Push, U1 STM32F405RGTx, U2 W25Q128JVP, U3 QMC5883P, U4 ICM-20602, U5 BMP580, U6 AP63205WU, U7 TLV75733PDBV, Y1 25MHz

Commit message: placement session: i am locked in
Parts:
- added D3: LED, LED_SMD:LED_0402_1005Metric, F.Cu at (152.1, 80.9)
- added D4: LED, LED_SMD:LED_0402_1005Metric, F.Cu at (152.1, 82.8)
- added D5: LED, LED_SMD:LED_0402_1005Metric, F.Cu at (152.1, 84.8)
- added R7: 1k, Resistor_SMD:R_0402_1005Metric, F.Cu at (149.0, 80.9)
- added R8: 220, Resistor_SMD:R_0402_1005Metric, F.Cu at (149.0, 82.8)
- added R9: 100, Resistor_SMD:R_0402_1005Metric, F.Cu at (149.0, 84.8)
- added TP21: TestPoint, nssfc:PAD_1.5mm, F.Cu at (167.9, 92.5)
- added TP22: TestPoint, nssfc:PAD_1.5mm, F.Cu at (167.9, 94.7)
- added TP23: TestPoint, nssfc:PAD_1.5mm, F.Cu at (167.9, 97.0)
- added TP24: TestPoint, nssfc:PAD_1.5mm, F.Cu at (167.9, 99.4)
- added TP25: TestPoint, nssfc:PAD_1.5mm, F.Cu at (179.7, 112.4)
- added TP26: TestPoint, nssfc:PAD_1.5mm, F.Cu at (182.2, 112.3)
- added TP27: TestPoint, nssfc:PAD_1.5mm, F.Cu at (200.9, 110.3)
- added TP28: TestPoint, nssfc:PAD_1.5mm, F.Cu at (200.8, 108.2)
- added TP29: TestPoint, nssfc:PAD_1.5mm, F.Cu at (200.8, 106.1)
- added TP30: TestPoint, nssfc:PAD_1.5mm, F.Cu at (200.9, 104.0)
- added TP31: TestPoint, nssfc:PAD_1.5mm, F.Cu at (167.9, 85.3)
- added TP32: TestPoint, nssfc:PAD_1.5mm, F.Cu at (167.9, 87.8)
- added TP33: TestPoint, nssfc:PAD_1.5mm, F.Cu at (167.8, 90.0)
- added TP34: TestPoint, nssfc:PAD_1.5mm, F.Cu at (183.7, 79.6)
- added TP35: TestPoint, nssfc:PAD_1.5mm, F.Cu at (167.9, 101.6)
- added TP36: TestPoint, nssfc:PAD_1.5mm, F.Cu at (167.9, 104.1)
- added TP37: TestPoint, nssfc:PAD_1.5mm, F.Cu at (167.9, 106.6)
- added TP38: TestPoint, nssfc:PAD_1.5mm, F.Cu at (200.9, 101.7)
- added TP39: TestPoint, nssfc:PAD_1.5mm, F.Cu at (200.9, 99.3)
- added TP40: TestPoint, nssfc:PAD_1.5mm, F.Cu at (200.9, 96.8)
- added TP41: TestPoint, nssfc:PAD_1.5mm, F.Cu at (184.5, 112.3)
- added TP42: TestPoint, nssfc:PAD_1.5mm, F.Cu at (187.1, 112.4)
- added TP43: TestPoint, nssfc:PAD_1.5mm, F.Cu at (189.6, 112.4)
- added TP44: TestPoint, nssfc:PAD_1.5mm, F.Cu at (181.5, 79.5)
- added TP45: TestPoint, nssfc:PAD_1.5mm, F.Cu at (179.2, 79.5)
- added TP46: TestPoint, nssfc:PAD_1.5mm, F.Cu at (176.7, 79.5)
- added TP47: TestPoint, nssfc:PAD_1.5mm, F.Cu at (167.8, 80.3)
- added TP48: TestPoint, nssfc:PAD_1.5mm, F.Cu at (167.8, 82.8)
- added TP49: TestPoint, nssfc:PAD_1.5mm, F.Cu at (191.8, 112.4)
- added TP50: TestPoint, TestPoint:TestPoint_Pad_3.0x3.0mm, F.Cu at (214.5, 79.4)
- added TP51: TestPoint, TestPoint:TestPoint_Pad_3.0x3.0mm, F.Cu at (214.5, 84.5)
- TP10, TP11, TP12, TP13, TP14, TP15, TP16, TP17, TP18, TP19, TP20, TP3, TP4, TP5, TP6, TP9: footprint TestPoint:TestPoint_Pad_1.5x1.5mm -> nssfc:PAD_1.5mm
- TP7, TP8: footprint TestPoint:TestPoint_Pad_1.5x1.5mm -> nssfc:PAD_1.5mm; moved to B.Cu
- moved R3 71.5 mm to (244.8, 97.5), turned to 0 degrees
- moved SW1 70.8 mm to (245.6, 89.7)
- moved TP8 68.0 mm to (180.2, 96.4), turned to 90 degrees
- moved C11 67.9 mm to (241.1, 94.0)
- moved R6 67.4 mm to (244.8, 103.4), turned to 0 degrees
- moved U2 65.6 mm to (238.4, 81.3), turned to 0 degrees
- moved C13 64.5 mm to (234.4, 105.4), turned to 0 degrees
- moved C21 63.0 mm to (241.1, 100.0), turned to 0 degrees
- moved U6 61.4 mm to (244.8, 80.5)
- moved C19 58.9 mm to (237.2, 107.4), turned to 0 degrees
- moved C16 57.7 mm to (234.4, 111.3), turned to 0 degrees
- moved C23 57.4 mm to (237.2, 109.4), turned to 0 degrees
- moved U7 56.4 mm to (244.8, 85.1)
- moved C7 56.2 mm to (231.5, 105.4)
- moved C22 55.7 mm to (241.1, 103.0)
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Connections:
- U1 pad 10: unconnected-(U1-PC2-Pad10) -> Net-(U1-PC2)
- U1 pad 11: unconnected-(U1-PC3-Pad11) -> Net-(U1-PC3)
- U1 pad 14: unconnected-(U1-PA0-Pad14) -> Net-(U1-PA0)
- U1 pad 15: unconnected-(U1-PA1-Pad15) -> Net-(U1-PA1)
- U1 pad 16: unconnected-(U1-PA2-Pad16) -> Net-(U1-PA2)
- U1 pad 2: unconnected-(U1-PC13-Pad2) -> Net-(U1-PC13)
- U1 pad 24: unconnected-(U1-PC4-Pad24) -> Net-(U1-PC4)
- U1 pad 25: unconnected-(U1-PC5-Pad25) -> Net-(U1-PC5)
- U1 pad 26: unconnected-(U1-PB0-Pad26) -> Net-(U1-PB0)
- U1 pad 27: unconnected-(U1-PB1-Pad27) -> Net-(U1-PB1)
- U1 pad 28: unconnected-(U1-PB2-Pad28) -> Net-(U1-PB2)
- U1 pad 29: unconnected-(U1-PB10-Pad29) -> Net-(U1-PB10)
- U1 pad 3: unconnected-(U1-PC14-Pad3) -> Net-(U1-PC14)
- U1 pad 37: unconnected-(U1-PC6-Pad37) -> Net-(U1-PC6)
- U1 pad 38: unconnected-(U1-PC7-Pad38) -> Net-(U1-PC7)
- U1 pad 39: unconnected-(U1-PC8-Pad39) -> Net-(U1-PC8)
- U1 pad 4: unconnected-(U1-PC15-Pad4) -> Net-(U1-PC15)
- U1 pad 40: unconnected-(U1-PC9-Pad40) -> Net-(U1-PC9)
- U1 pad 41: unconnected-(U1-PA8-Pad41) -> Net-(U1-PA8)
- U1 pad 42: unconnected-(U1-PA9-Pad42) -> Net-(U1-PA9)
- U1 pad 43: unconnected-(U1-PA10-Pad43) -> Net-(U1-PA10)
- U1 pad 54: unconnected-(U1-PD2-Pad54) -> Net-(U1-PD2)
- U1 pad 55: unconnected-(U1-PB3-Pad55) -> Net-(U1-PB3)
- U1 pad 56: unconnected-(U1-PB4-Pad56) -> Net-(U1-PB4)
- U1 pad 57: unconnected-(U1-PB5-Pad57) -> Net-(U1-PB5)
- U1 pad 61: unconnected-(U1-PB8-Pad61) -> Net-(U1-PB8)
- U1 pad 62: unconnected-(U1-PB9-Pad62) -> Net-(U1-PB9)
- U1 pad 8: unconnected-(U1-PC0-Pad8) -> Net-(U1-PC0)
- U1 pad 9: unconnected-(U1-PC1-Pad9) -> Net-(U1-PC1)
Routing:
- net +3V3: track 55.5 -> 0.00 mm, vias 4 -> 0
- net Net-(U1-BOOT0): track 22.8 -> 0.00 mm, vias 2 -> 0
- net /IMU_SPI_CS: track 20.4 -> 0.00 mm, vias 2 -> 0
- net /IMU_SPI_SCK: track 19.6 -> 0.00 mm
- net /IMU_SPI_MOSI: track 19.4 -> 0.00 mm, vias 2 -> 0
- net Net-(D2-A): track 17.7 -> 0.00 mm
- net /IMU_SPI_MISO: track 16.6 -> 0.00 mm, vias 2 -> 0
- net GND: track 13.4 -> 0.00 mm, vias 11 -> 0
- net Net-(D1-A): track 12.0 -> 0.00 mm
- net /F_SPI_MOSI: track 11.5 -> 0.00 mm, vias 2 -> 0
- net +5V: track 11.3 -> 0.00 mm
- net /F_SPI_CLK: track 10.3 -> 0.00 mm, vias 2 -> 0
- net /M_SCK: track 10.3 -> 0.00 mm, vias 2 -> 0
- net /~{F_SPI_WP}: track 10.3 -> 0.00 mm
- net VBUS: track 9.38 -> 0.00 mm, vias 2 -> 0
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
Commit message: completed placement
Parts:
- removed C18: 10n, Capacitor_SMD:C_0402_1005Metric
- removed TP10, TP11, TP12, TP13, TP14, TP15, TP16, TP17, TP18, TP19, TP20, TP3, TP4, TP5, TP6, TP7, TP8, TP9: TestPoint, nssfc:PAD_1.5mm
- added TP52: TestPoint, nssfc:PAD_1.5mm, F.Cu at (167.8, 92.1)
- added TP53: TestPoint, nssfc:PAD_1.5mm, F.Cu at (200.9, 95.0)
- added TP55: TestPoint, nssfc:PAD_1.5mm, F.Cu at (192.7, 112.4)
- added TP58: TestPoint, nssfc:PAD_1.5mm, F.Cu at (195.2, 112.4)
- added TP59: TestPoint, nssfc:PAD_1.5mm, F.Cu at (167.8, 94.3)
- added TP60: TestPoint, nssfc:PAD_1.5mm, F.Cu at (175.7, 112.4)
- added TP61: TestPoint, nssfc:PAD_1.5mm, F.Cu at (188.2, 79.3)
- added TP62: TestPoint, nssfc:PAD_1.5mm, F.Cu at (190.6, 79.3)
- added TP63: TestPoint, nssfc:PAD_1.5mm, F.Cu at (173.3, 112.4)
- added TP64: TestPoint, nssfc:PAD_1.5mm, F.Cu at (200.9, 97.0)
- TP1, TP2: moved to B.Cu
- TP50, TP51: footprint TestPoint:TestPoint_Pad_3.0x3.0mm -> TestPoint:TestPoint_Pad_2.0x2.0mm; moved to B.Cu
- moved TP1 80.6 mm to (171.4, 101.8), turned to 180 degrees
- moved TP2 80.6 mm to (171.4, 104.9), turned to 180 degrees
- moved R3 77.5 mm to (169.3, 79.9), turned to 90 degrees
- moved R2 75.5 mm to (171.3, 77.9), turned to 180 degrees
- moved R1 74.8 mm to (170.9, 104.9)
- moved U4 74.5 mm to (174.9, 108.3), turned to 180 degrees
- moved U7 73.8 mm to (171.5, 93.2), turned to -90 degrees
- moved C22 70.8 mm to (171.4, 90.2), turned to 180 degrees
- moved U6 70.2 mm to (174.8, 85.2)
- moved C24 69.7 mm to (172.0, 96.3), turned to 180 degrees
- moved C11 67.6 mm to (174.6, 81.7), turned to -90 degrees
- moved C21 67.3 mm to (174.8, 87.9)
- moved C23 66.3 mm to (173.6, 90.6), turned to 90 degrees
- moved C25 65.8 mm to (173.7, 94.2), turned to 90 degrees
- moved SW1 64.8 mm to (181.1, 83.6)
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Routing:
- net /M_SDA: track 0.00 -> 26.6 mm, vias 0 -> 2
- net /M_SCK: track 0.00 -> 24.4 mm, vias 0 -> 2
- net /~{F_SPI_WP}: track 0.00 -> 15.4 mm, vias 0 -> 2
- net /IMU_SPI_SCK: track 0.00 -> 12.9 mm
- net /~{F_SPI_CS}: track 0.00 -> 12.0 mm, vias 0 -> 2
- net /BMP_SPI_SCK: track 0.00 -> 11.4 mm, vias 0 -> 2
- net /IMU_SPI_MOSI: track 0.00 -> 10.4 mm
- net /F_SPI_MISO: track 0.00 -> 9.96 mm, vias 0 -> 2
- net /BMP_SPI_INT: track 0.00 -> 9.83 mm
- net /IMU_SPI_MISO: track 0.00 -> 9.69 mm
- net /IMU_SPI_CS: track 0.00 -> 8.49 mm
- net /BMP_SPI_MOSI: track 0.00 -> 7.95 mm
- net /BMP_SPI_MISO: track 0.00 -> 7.20 mm
- net /BMP_SPI_CSB: track 0.00 -> 6.76 mm
- net /IMU_SPI_INT: track 0.00 -> 6.31 mm
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- added copper zone on In1.Cu, net GND

Commit message: Completed PCB
Parts:
- moved TP55 2.45 mm to (195.2, 112.4)
- moved TP58 2.44 mm to (192.7, 112.4)
- moved R6 1.12 mm to (182.1, 91.6), turned to 180 degrees
- moved C7 0.07 mm to (180.7, 106.7)
Routing:
- net +5V: track 0.00 -> 60.3 mm, vias 0 -> 3
- net +3V3: track 0.00 -> 49.0 mm, vias 0 -> 15
- net VBUS: track 0.00 -> 31.1 mm, vias 0 -> 2
- net Net-(U1-PB8): track 0.00 -> 21.9 mm, vias 0 -> 2
- net Net-(U1-PB9): track 0.00 -> 20.1 mm, vias 0 -> 2
- net Net-(U1-PB3): track 0.00 -> 19.2 mm, vias 0 -> 2
- net Net-(U1-PC14): track 0.00 -> 18.6 mm, vias 0 -> 2
- net /NRST: track 0.00 -> 18.5 mm, vias 0 -> 2
- net Net-(U1-PB4): track 0.00 -> 18.1 mm, vias 0 -> 2
- net Net-(U1-PC15): track 0.00 -> 17.9 mm, vias 0 -> 2
- net Net-(U1-PC13): track 0.00 -> 17.8 mm, vias 0 -> 2
- net /USB_DP: track 0.00 -> 17.7 mm
- net /USB_DN: track 0.00 -> 17.6 mm
- net Net-(U1-PD2): track 0.00 -> 17.6 mm, vias 0 -> 2
- net Net-(U1-PB5): track 0.00 -> 17.4 mm, vias 0 -> 2
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- added copper zone on In2.Cu, net +3V3
- added copper zone on In2.Cu, net GND
- removed copper zone on In1.Cu, net GND
