File: hardware/nssfc.kicad_pcb (KiCad board)
At the start: 4 copper layers, 37 x 37 mm, 92 parts, among them J1 USB_C_Receptacle_USB2.0_16P, SW1 SW_Push, U1 STM32F405RGTx, U2 W25Q128JVP, U3 QMC5883P, U4 ICM-20602, U5 BMP580, U6 AP63205WU, U7 TLV75733PDBV, Y1 25MHz

Commit message: done PCB
Parts:
- added G***: LOGO, LOGO, F.Cu at (196.0, 100.1)
- moved R3 1.04 mm to (169.1, 78.9), turned to -90 degrees
- moved C17 0.94 mm to (177.4, 109.2)
- moved C15 0.94 mm to (171.9, 109.7)
- moved C16 0.94 mm to (175.8, 109.7)
- moved U4 0.94 mm to (174.9, 107.4)
- moved TP27 0.83 mm to (201.4, 110.4)
- moved TP39 0.83 mm to (201.5, 100.4)
- moved TP40 0.83 mm to (201.5, 98.4)
- moved TP28 0.83 mm to (201.4, 108.4)
- moved TP29 0.83 mm to (201.4, 106.4)
- moved TP30 0.83 mm to (201.4, 104.4)
- moved TP38 0.83 mm to (201.4, 102.4)
- moved TP53 0.83 mm to (201.5, 94.4)
- moved TP64 0.83 mm to (201.5, 96.4)
- moved TP34 0.70 mm to (185.8, 78.6)
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Routing:
- net +3V3: track 49.0 -> 26.7 mm, vias 15 -> 17
- net +5V: track 60.3 -> 56.7 mm, vias 3 -> 4
- net Net-(U6-SW): track 3.77 -> 0.27 mm
- net /~{F_SPI_CS}: track 12.0 -> 9.64 mm
- net Net-(D2-A): track 15.3 -> 13.3 mm
- net Net-(U1-PB4): track 18.1 -> 16.5 mm
- net Net-(U1-PB3): track 19.2 -> 20.6 mm
- net VBUS: track 31.1 -> 32.1 mm, vias 2 -> 3
- net Net-(U1-PD2): track 17.6 -> 18.5 mm
- net GND: track 15.3 -> 14.7 mm, vias 19 -> 27
- added copper zone on F.Cu, net +3V3
- added copper zone on F.Cu, net +5V
- added copper zone on In1.Cu, net GND
- added copper zone on F.Cu, net Net-(U6-SW)
- removed copper zone on In2.Cu, net GND
Other:
- board text added: "3V3"
- board text added: "5V"
- board text added: "GND"
- board text added: "Made by Keyaan and Ahad"
- board text added: "PA0"
- board text added: "PA1"
- board text added: "PA10"
- board text added: "PA2"
- board text added: "PA8"
- board text added: "PA9"
- board text added: "PB0"
- board text added: "PB1"
- board text added: "PB10"
- board text added: "PB2"
- board text added: "PB3"
- board text added: "PB4"
- board text added: "PB5"
- board text added: "PB8"
- board text added: "PB9"
- board text added: "PC0"
- board text added: "PC1"
- board text added: "PC14"
- board text added: "PC15"
- board text added: "PC2"
- board text added: "PC3"
- board text added: "PC4"
- board text added: "PC5"
- board text added: "PC6"
- board text added: "PC7"
- board text added: "PC8"
- board text added: "PC9"
- board text added: "VBUS"
