File: hardware/nssfc.kicad_pcb (KiCad board)
At the start: 4 copper layers, 37 x 37 mm, 92 parts, among them J1 USB_C_Receptacle_USB2.0_16P, SW1 SW_Push, U1 STM32F405RGTx, U2 W25Q128JVP, U3 QMC5883P, U4 ICM-20602, U5 BMP580, U6 AP63205WU, U7 TLV75733PDBV, Y1 25MHz

Commit message: Rerouted PCB
Parts:
- added H1: MountingHole, MountingHole:MountingHole_3.2mm_M3, F.Cu at (169.7, 80.6)
- added H2: MountingHole, MountingHole:MountingHole_3.2mm_M3, F.Cu at (199.5, 110.3)
- added H3: MountingHole, MountingHole:MountingHole_3.2mm_M3, F.Cu at (169.8, 110.4)
- added H4: MountingHole, MountingHole:MountingHole_3.2mm_M3, F.Cu at (199.3, 80.5)
- TP52, TP55, TP58, TP60, TP61, TP62, TP64: moved to B.Cu
- moved TP60 35.6 mm to (185.4, 78.2), turned to 180 degrees
- moved TP59 34.8 mm to (201.9, 101.5), turned to 0 degrees
- moved TP52 34.4 mm to (201.9, 96.8), turned to 180 degrees
- moved TP61 33.5 mm to (188.8, 112.8), turned to 180 degrees
- moved TP62 33.5 mm to (191.2, 112.8), turned to 180 degrees
- moved C22 32.1 mm to (199.9, 105.0), turned to 90 degrees
- moved TP58 30.7 mm to (167.3, 95.2), turned to 180 degrees
- moved J1 29.9 mm to (178.6, 110.1), turned to 0 degrees
- moved TP63 29.3 mm to (201.9, 106.1)
- moved C19 29.2 mm to (192.9, 109.3)
- moved U6 29.0 mm to (190.3, 109.8)
- moved R7 28.9 mm to (183.6, 104.3), turned to -90 degrees
- moved TP51 28.3 mm to (167.8, 101.3), turned to 180 degrees
- moved C13 27.9 mm to (179.1, 86.3)
- moved C24 27.7 mm to (199.1, 102.3)
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Routing:
- net +5V: track 60.3 -> 38.9 mm, vias 3 -> 2
- net /M_SDA: track 26.6 -> 7.96 mm
- net /M_SCK: track 24.4 -> 7.58 mm, vias 2 -> 0
- net +3V3: track 49.0 -> 65.5 mm, vias 15 -> 10
- net Net-(U1-PB10): track 9.33 -> 23.0 mm, vias 0 -> 2
- net Net-(U1-PB1): track 7.92 -> 20.6 mm, vias 0 -> 2
- net Net-(U1-PB2): track 8.53 -> 20.7 mm, vias 0 -> 2
- net Net-(U1-PB0): track 8.72 -> 20.4 mm, vias 0 -> 2
- net GND: track 15.3 -> 26.2 mm, vias 19 -> 11
- net /USB_DN: track 17.8 -> 28.5 mm, vias 0 -> 2
- net Net-(U1-PC5): track 9.52 -> 20.1 mm, vias 0 -> 2
- net Net-(U1-PA2): track 13.9 -> 24.5 mm, vias 0 -> 2
- net Net-(U1-PC4): track 10.6 -> 19.7 mm, vias 0 -> 2
- net /USB_DP: track 17.8 -> 25.4 mm, vias 0 -> 2
- net Net-(U1-PB8): track 21.9 -> 14.5 mm
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- added copper zone on In1.Cu, net GND
- removed copper zone on In2.Cu, net GND

Commit message: done
Parts:
- added G***: LOGO, LOGO, F.Cu at (172.8, 96.5)
