File: hardware/nssfc.kicad_sch (KiCad schematic)
At the start: 92 parts, among them J1 USB_C_Receptacle_USB2.0_16P, SW1 SW_Push, U1 STM32F405RGTx, U2 W25Q128JVP, U3 QMC5883P, U4 ICM-20602, U5 BMP580, U6 AP63205WU, U7 TLV75733PDBV, Y1 25MHz

Commit message: Rerouted PCB
Parts:
- added H1, H2, H3, H4: MountingHole, MountingHole:MountingHole_3.2mm_M3, symbol Mechanical:MountingHole
